File: tester.sch (KiCad schematic (older format))
At the start: 15 parts

Commit message: next step
Parts:
- removed BUZ1: BUZZER, symbol BUZZER
- added BZ1: BUZZER, ~, symbol BUZZER
- DA1: value GIC_OPAMP_UD608 -> УД608; footprint (none) -> ~
Changed lines of the file:
@@
 LIBS:conn
 LIBS:mixture
+LIBS:tester-cache
 EELAYER 27 0
 EELAYER END
@@
 $EndDescr
 $Comp
-L GIC_OPAMP_UD608 DA1
-U 1 1 530321E0
-P 7250 2650
-F 0 "DA1" H 7750 2800 60  0000 C CNN
-F 1 "GIC_OPAMP_UD608" H 7750 2100 60  0000 C CNN
-F 2 "" H 7250 2650 60  0000 C CNN
-F 3 "" H 7250 2650 60  0000 C CNN
-	1    7250 2650
-	1    0    0    -1
-$EndComp
-$Comp
 L RES R1
 U 1 1 530321EF
@@
 $EndComp
 $Comp
-L POWER_GND #~01
+L POWER_GND #01
 U 1 1 530322A3
 P 4550 5700
-F 0 "#~01" V 4500 5650 60  0001 C CNN
+F 0 "#01" V 4500 5650 60  0001 C CNN
 F 1 "POWER_GND" V 4600 5650 60  0001 C CNN
 F 2 "" H 4550 5700 60  0000 C CNN
@@
 $EndComp
 $Comp
-L POWER_GND #~02
+L POWER_GND #02
 U 1 1 5303463F
 P 5750 2100
-F 0 "#~02" V 5700 2050 60  0001 C CNN
+F 0 "#02" V 5700 2050 60  0001 C CNN
 F 1 "POWER_GND" V 5800 2050 60  0001 C CNN
 F 2 "" H 5750 2100 60  0000 C CNN
@@
 $EndComp
 $Comp
-L POWER_GND #~03
+L POWER_GND #03
 U 1 1 530346AA
 P 6100 3850
-F 0 "#~03" V 6050 3800 60  0001 C CNN
+F 0 "#03" V 6050 3800 60  0001 C CNN
 F 1 "POWER_GND" V 6150 3800 60  0001 C CNN
 F 2 "" H 6100 3850 60  0000 C CNN
@@
 $EndComp
 $Comp
-L POWER_GND #~04
+L POWER_GND #04
 U 1 1 53034A91
 P 8900 3850
-F 0 "#~04" V 8850 3800 60  0001 C CNN
+F 0 "#04" V 8850 3800 60  0001 C CNN
 F 1 "POWER_GND" V 8950 3800 60  0001 C CNN
 F 2 "" H 8900 3850 60  0000 C CNN
@@
 $EndComp
 $Comp
-L POWER_GND #~05
+L POWER_GND #05
 U 1 1 53034BFE
 P 8400 3150
-F 0 "#~05" V 8350 3100 60  0001 C CNN
+F 0 "#05" V 8350 3100 60  0001 C CNN
 F 1 "POWER_GND" V 8450 3100 60  0001 C CNN
 F 2 "" H 8400 3150 60  0000 C CNN
@@
 	1    0    0    -1
 $EndComp
-$Comp
-L BUZZER BUZ1
-U 1 1 53035F9F
-P 9100 3650
-F 0 "BUZ1" H 9200 3950 60  0000 C CNN
-F 1 "BUZZER" H 9200 3550 60  0000 C CNN
-F 2 "" H 9100 3650 60  0000 C CNN
-F 3 "" H 9100 3650 60  0000 C CNN
-	1    9100 3650
-	1    0    0    -1
-$EndComp
 Wire Wire Line
 	8250 2650 8900 2650
@@
 Connection ~ 4550 3500
 Wire Wire Line
-	8900 3450 8900 3500
-Wire Wire Line
-	8900 3500 9000 3500
-Wire Wire Line
-	9000 3600 8900 3600
-Wire Wire Line
-	8900 3600 8900 3850
-Wire Wire Line
 	4550 2850 6250 2850
 Connection ~ 5250 2850
@@
 	5250 4450 5250 4250
 Wire Wire Line
-	7350 2100 6650 2100
-Wire Wire Line
-	7350 3650 7000 3650
+	6650 2100 7350 2100
+Wire Wire Line
+	7000 3650 7350 3650
 Wire Wire Line
 	7250 2650 7150 2650
@@
 	4900 2750 4900 2850
 Connection ~ 4900 2850
+Wire Wire Line
+	8900 3450 8900 3550
+$Comp
+L GIC_OPAMP_UD608 DA1
+U 1 1 53036D18
+P 7250 2650
+F 0 "DA1" H 7750 2800 60  0000 C CNN
+F 1 "УД608" H 7750 2100 60  0000 C CNN
+F 2 "~" H 7250 2650 60  0000 C CNN
+F 3 "~" H 7250 2650 60  0000 C CNN
+	1    7250 2650
+	1    0    0    -1
+$EndComp
+$Comp
+L BUZZER BZ1
+U 1 1 53038C16
+P 9300 3650
+F 0 "BZ1" H 9200 3900 70  0000 C CNN
+F 1 "BUZZER" H 9200 3400 70  0000 C CNN
+F 2 "~" H 9300 3650 60  0000 C CNN
+F 3 "~" H 9300 3650 60  0000 C CNN
+	1    9300 3650
+	1    0    0    -1
+$EndComp
+Wire Wire Line
+	8900 3550 9050 3550
+Wire Wire Line
+	9050 3750 8900 3750
+Wire Wire Line
+	8900 3750 8900 3850
 $EndSCHEMATC

Commit message: changes
Parts:
- removed R6: RES, symbol RES
- removed VD1: DIODE_LIGHT, symbol DIODE_LIGHT
- renumbered R7 to R6, VD2 to VD1
Changed lines of the file:
@@
 $EndComp
 $Comp
-L RES R7
+L RES R6
 U 1 1 53032285
 P 5250 4450
-F 0 "R7" H 5500 4575 60  0000 C CNN
+F 0 "R6" H 5500 4575 60  0000 C CNN
 F 1 "RES" H 5750 4575 60  0000 C CNN
 F 2 "" H 5250 4450 60  0000 C CNN
@@
 $EndComp
 $Comp
-L DIODE_LIGHT VD1
-U 1 1 530343A0
-P 3900 3650
-F 0 "VD1" H 4250 3950 60  0000 C CNN
-F 1 "DIODE_LIGHT" H 4250 3400 60  0000 C CNN
-F 2 "" H 3900 3650 60  0000 C CNN
-F 3 "" H 3900 3650 60  0000 C CNN
-	1    3900 3650
-	0    -1   1    0
-$EndComp
-$Comp
 L POWER_GND #02
 U 1 1 5303463F
@@
 $EndComp
 $Comp
-L DIODE_LIGHT VD2
+L DIODE_LIGHT VD1
 U 1 1 5303476E
 P 5250 3650
-F 0 "VD2" H 5600 3950 60  0000 C CNN
+F 0 "VD1" H 5600 3950 60  0000 C CNN
 F 1 "DIODE_LIGHT" H 5600 3400 60  0000 C CNN
 F 2 "" H 5250 3650 60  0000 C CNN
 F 3 "" H 5250 3650 60  0000 C CNN
 	1    5250 3650
-	0    -1   1    0
-$EndComp
-$Comp
-L RES R6
-U 1 1 5303477A
-P 3900 4450
-F 0 "R6" H 4150 4575 60  0000 C CNN
-F 1 "RES" H 4400 4575 60  0000 C CNN
-F 2 "" H 3900 4450 60  0000 C CNN
-F 3 "" H 3900 4450 60  0000 C CNN
-	1    3900 4450
 	0    -1   1    0
 $EndComp
@@
 	1    0    0    -1
 $EndComp
-Wire Wire Line
-	8250 2650 8900 2650
-Wire Wire Line
-	8150 2100 8650 2100
-Wire Wire Line
-	7150 2650 7150 2100
-Wire Wire Line
-	6200 2100 5750 2100
-Wire Wire Line
-	7050 2850 7250 2850
-Wire Wire Line
-	7150 2850 7150 3650
-Connection ~ 7150 3650
-Connection ~ 7150 2850
-Wire Wire Line
-	6200 3650 6100 3650
-Wire Wire Line
-	6100 3650 6100 3850
-Wire Wire Line
-	3900 5600 3900 5250
-Connection ~ 4550 5600
-Wire Wire Line
-	3900 3650 3900 3500
-Wire Wire Line
-	4550 4350 4550 4250
-Wire Wire Line
-	5250 5600 5250 5250
-Wire Wire Line
-	3900 5600 5250 5600
-Wire Wire Line
-	4550 4800 4550 5700
-Connection ~ 4550 3500
-Wire Wire Line
-	4550 2850 6250 2850
-Connection ~ 5250 2850
-Wire Wire Line
-	8250 3050 8400 3050
-Wire Wire Line
-	8400 3050 8400 3150
-Wire Wire Line
-	8650 3650 8150 3650
-Wire Wire Line
-	8650 2100 8650 3650
-Connection ~ 8650 2650
-Wire Wire Line
-	3900 4450 3900 4250
-Wire Wire Line
-	4550 3150 4550 3850
-Wire Wire Line
-	4550 3050 4550 2850
-Wire Wire Line
-	5250 4450 5250 4250
-Wire Wire Line
-	6650 2100 7350 2100
-Wire Wire Line
-	7000 3650 7350 3650
-Wire Wire Line
-	7250 2650 7150 2650
-Connection ~ 7150 2100
-Connection ~ 3900 3500
-Wire Wire Line
-	3900 3500 4550 3500
-Wire Wire Line
-	8250 2850 8400 2850
-Wire Wire Line
-	8400 2850 8400 2350
-Wire Wire Line
-	8400 2350 5250 2350
-Wire Wire Line
-	5250 2350 5250 3650
 $Comp
 L PWR_FLAG #FLG06
-U 1 1 530388A3
-P 4350 5400
-F 0 "#FLG06" H 4350 5495 30  0001 C CNN
-F 1 "PWR_FLAG" H 4350 5580 30  0000 C CNN
-F 2 "" H 4350 5400 60  0000 C CNN
-F 3 "" H 4350 5400 60  0000 C CNN
-	1    4350 5400
-	1    0    0    -1
-$EndComp
-Wire Wire Line
-	4350 5400 4550 5400
-Connection ~ 4550 5400
-$Comp
-L PWR_FLAG #FLG07
 U 1 1 53038977
 P 4900 2750
-F 0 "#FLG07" H 4900 2845 30  0001 C CNN
+F 0 "#FLG06" H 4900 2845 30  0001 C CNN
 F 1 "PWR_FLAG" H 4900 2930 30  0000 C CNN
 F 2 "" H 4900 2750 60  0000 C CNN
@@
 	1    0    0    -1
 $EndComp
-Wire Wire Line
-	4900 2750 4900 2850
-Connection ~ 4900 2850
-Wire Wire Line
-	8900 3450 8900 3550
 $Comp
 L GIC_OPAMP_UD608 DA1
@@
 	1    0    0    -1
 $EndComp
+Wire Wire Line
+	8250 2650 8900 2650
+Wire Wire Line
+	8150 2100 8650 2100
+Wire Wire Line
+	7150 2650 7150 2100
+Wire Wire Line
+	6200 2100 5750 2100
+Wire Wire Line
+	7050 2850 7250 2850
+Wire Wire Line
+	7150 2850 7150 3650
+Connection ~ 7150 3650
+Connection ~ 7150 2850
+Wire Wire Line
+	6200 3650 6100 3650
+Wire Wire Line
+	6100 3650 6100 3850
+Wire Wire Line
+	4550 4350 4550 4250
+Wire Wire Line
+	4550 4800 4550 5700
+Connection ~ 4550 3500
+Wire Wire Line
+	4550 2850 6250 2850
+Connection ~ 5250 2850
+Wire Wire Line
+	8250 3050 8400 3050
+Wire Wire Line
+	8400 3050 8400 3150
+Wire Wire Line
+	8650 3650 8150 3650
+Wire Wire Line
+	8650 2100 8650 3650
+Connection ~ 8650 2650
+Wire Wire Line
+	4550 3150 4550 3850
+Wire Wire Line
+	4550 3050 4550 2850
+Wire Wire Line
+	5250 4450 5250 4250
+Wire Wire Line
+	6650 2100 7350 2100
+Wire Wire Line
+	7000 3650 7350 3650
+Wire Wire Line
+	7250 2650 7150 2650
+Connection ~ 7150 2100
+Wire Wire Line
+	8250 2850 8400 2850
+Wire Wire Line
+	8400 2850 8400 2350
+Wire Wire Line
+	8400 2350 5250 2350
+Wire Wire Line
+	5250 2350 5250 3650
+Wire Wire Line
+	4900 2750 4900 2850
+Connection ~ 4900 2850
+Wire Wire Line
+	8900 3700 8900 3850
+Wire Wire Line
+	5250 5600 5250 5250
+Connection ~ 4550 5400
+Connection ~ 4550 5600
+Wire Wire Line
+	4350 5400 4550 5400
+$Comp
+L PWR_FLAG #FLG07
+U 1 1 530388A3
+P 4350 5400
+F 0 "#FLG07" H 4350 5495 30  0001 C CNN
+F 1 "PWR_FLAG" H 4350 5580 30  0000 C CNN
+F 2 "" H 4350 5400 60  0000 C CNN
+F 3 "" H 4350 5400 60  0000 C CNN
+	1    4350 5400
+	1    0    0    -1
+$EndComp
+Wire Wire Line
+	5250 5600 4550 5600
 $Comp
 L BUZZER BZ1
-U 1 1 53038C16
-P 9300 3650
-F 0 "BZ1" H 9200 3900 70  0000 C CNN
-F 1 "BUZZER" H 9200 3400 70  0000 C CNN
-F 2 "~" H 9300 3650 60  0000 C CNN
-F 3 "~" H 9300 3650 60  0000 C CNN
-	1    9300 3650
-	1    0    0    -1
-$EndComp
-Wire Wire Line
-	8900 3550 9050 3550
-Wire Wire Line
-	9050 3750 8900 3750
-Wire Wire Line
-	8900 3750 8900 3850
+U 1 1 5303A8D4
+P 9150 3600
+F 0 "BZ1" H 9050 3850 70  0000 C CNN
+F 1 "BUZZER" H 9050 3350 70  0000 C CNN
+F 2 "~" H 9150 3600 60  0000 C CNN
+F 3 "~" H 9150 3600 60  0000 C CNN
+	1    9150 3600
+	1    0    0    -1
+$EndComp
+Wire Wire Line
+	8900 3500 8900 3450
 $EndSCHEMATC

Commit message: next step
Parts:
- C1: value CAP -> 0,1
- GB1: value BAT -> 3В
- R1, R2: value RES -> 5,1K
- R3: value RES -> 1,8K
- R4: value RES -> 3,6K
- R5: value RES -> 50
- R6: value RES -> 100
Other:
- moved on the sheet: GB1, R3, R6, SA1, VD1, XS1
Changed lines of the file:
@@
 Sheet 1 1
 Title ""
-Date "18 feb 2014"
+Date "28 feb 2014"
 Rev ""
 Comp ""
@@
 P 7350 2100
 F 0 "R1" H 7600 2225 60  0000 C CNN
-F 1 "RES" H 7850 2225 60  0000 C CNN
+F 1 "5,1K" H 7600 1950 60  0000 C CNN
 F 2 "" H 7350 2100 60  0000 C CNN
 F 3 "" H 7350 2100 60  0000 C CNN
@@
 L RES R3
 U 1 1 5303220D
-P 6200 3650
-F 0 "R3" H 6450 3775 60  0000 C CNN
-F 1 "RES" H 6700 3775 60  0000 C CNN
-F 2 "" H 6200 3650 60  0000 C CNN
-F 3 "" H 6200 3650 60  0000 C CNN
-	1    6200 3650
-	1    0    0    -1
+P 7000 4500
+F 0 "R3" V 7600 4350 60  0000 C CNN
+F 1 "1,8K" V 7250 4250 60  0000 C CNN
+F 2 "" H 7000 4500 60  0000 C CNN
+F 3 "" H 7000 4500 60  0000 C CNN
+	1    7000 4500
+	0    -1   -1   0
 $EndComp
 $Comp
@@
 P 6250 2850
 F 0 "R4" H 6500 2975 60  0000 C CNN
-F 1 "RES" H 6750 2975 60  0000 C CNN
+F 1 "3,6K" H 6550 2700 60  0000 C CNN
 F 2 "" H 6250 2850 60  0000 C CNN
 F 3 "" H 6250 2850 60  0000 C CNN
@@
 U 1 1 5303222B
 P 6200 2100
-F 0 "C1" H 6350 2000 60  0000 C CNN
-F 1 "CAP" H 6375 1750 60  0000 C CNN
+F 0 "C1" V 6350 1750 60  0000 C CNN
+F 1 "0,1" V 6100 1750 60  0000 C CNN
 F 2 "" H 6200 2100 60  0000 C CNN
 F 3 "" H 6200 2100 60  0000 C CNN
@@
 L BAT GB1
 U 1 1 5303223A
-P 4550 4350
-F 0 "GB1" H 4575 4225 60  0000 L CNN
-F 1 "BAT" H 4575 4025 60  0000 L CNN
-F 2 "" H 4550 4350 60  0000 C CNN
-F 3 "" H 4550 4350 60  0000 C CNN
-	1    4550 4350
+P 5400 3800
+F 0 "GB1" H 5425 3675 60  0000 L CNN
+F 1 "3В" H 5425 3475 60  0000 L CNN
+F 2 "" H 5400 3800 60  0000 C CNN
+F 3 "" H 5400 3800 60  0000 C CNN
+	1    5400 3800
 	-1   0    0    -1
 $EndComp
@@
 L CONN_02_F XS1
 U 1 1 53032249
-P 4550 3050
-F 0 "XS1" H 4800 3150 60  0000 C CNN
-F 1 "CONN_02_F" H 4900 2850 60  0000 C CNN
-F 2 "" H 4550 3050 60  0000 C CNN
-F 3 "" H 4550 3050 60  0000 C CNN
-	1    4550 3050
+P 5400 3050
+F 0 "XS1" H 5650 3150 60  0000 C CNN
+F 1 "CONN_02_F" H 5750 2850 60  0001 C CNN
+F 2 "" H 5400 3050 60  0000 C CNN
+F 3 "" H 5400 3050 60  0000 C CNN
+	1    5400 3050
 	-1   0    0    -1
 $EndComp
@@
 P 7350 3650
 F 0 "R2" H 7600 3775 60  0000 C CNN
-F 1 "RES" H 7850 3775 60  0000 C CNN
+F 1 "5,1K" H 7650 3500 60  0000 C CNN
 F 2 "" H 7350 3650 60  0000 C CNN
 F 3 "" H 7350 3650 60  0000 C CNN
@@
 L RES R6
 U 1 1 53032285
-P 5250 4450
-F 0 "R6" H 5500 4575 60  0000 C CNN
-F 1 "RES" H 5750 4575 60  0000 C CNN
-F 2 "" H 5250 4450 60  0000 C CNN
-F 3 "" H 5250 4450 60  0000 C CNN
-	1    5250 4450
+P 6100 3900
+F 0 "R6" V 6350 3750 60  0000 C CNN
+F 1 "100" V 6650 3700 60  0000 C CNN
+F 2 "" H 6100 3900 60  0000 C CNN
+F 3 "" H 6100 3900 60  0000 C CNN
+	1    6100 3900
 	0    -1   1    0
 $EndComp
@@
 U 1 1 53032294
 P 8900 2650
-F 0 "R5" H 9150 2775 60  0000 C CNN
-F 1 "RES" H 9400 2775 60  0000 C CNN
+F 0 "R5" V 9150 2800 60  0000 C CNN
+F 1 "50" V 9450 2800 60  0000 C CNN
 F 2 "" H 8900 2650 60  0000 C CNN
 F 3 "" H 8900 2650 60  0000 C CNN
@@
 L POWER_GND #01
 U 1 1 530322A3
-P 4550 5700
-F 0 "#01" V 4500 5650 60  0001 C CNN
-F 1 "POWER_GND" V 4600 5650 60  0001 C CNN
-F 2 "" H 4550 5700 60  0000 C CNN
-F 3 "" H 4550 5700 60  0000 C CNN
-	1    4550 5700
+P 5400 4800
+F 0 "#01" V 5350 4750 60  0001 C CNN
+F 1 "POWER_GND" V 5450 4750 60  0001 C CNN
+F 2 "" H 5400 4800 60  0000 C CNN
+F 3 "" H 5400 4800 60  0000 C CNN
+	1    5400 4800
 	-1   0    0    -1
 $EndComp
@@
 L SA_1-2_CL SA1
 U 1 1 530322B2
-P 4550 4050
-F 0 "SA1" H 4550 4250 120 0000 C CNN
-F 1 "SA_1-2_CL" H 4550 3950 60  0000 C CNN
-F 2 "~" H 4550 4050 60  0000 C CNN
-F 3 "~" H 4550 4050 60  0000 C CNN
-	1    4550 4050
+P 5400 3500
+F 0 "SA1" V 5450 3350 59  0000 C CNN
+F 1 "SA_1-2_CL" H 5400 3300 60  0001 C CNN
+F 2 "~" H 5400 3500 60  0000 C CNN
+F 3 "~" H 5400 3500 60  0000 C CNN
+	1    5400 3500
 	0    1    -1   0
 $EndComp
@@
 L POWER_GND #02
 U 1 1 5303463F
-P 5750 2100
-F 0 "#02" V 5700 2050 60  0001 C CNN
-F 1 "POWER_GND" V 5800 2050 60  0001 C CNN
-F 2 "" H 5750 2100 60  0000 C CNN
-F 3 "" H 5750 2100 60  0000 C CNN
-	1    5750 2100
+P 5100 2100
+F 0 "#02" V 5050 2050 60  0001 C CNN
+F 1 "POWER_GND" V 5150 2050 60  0001 C CNN
+F 2 "" H 5100 2100 60  0000 C CNN
+F 3 "" H 5100 2100 60  0000 C CNN
+	1    5100 2100
 	-1   0    0    -1
 $EndComp
@@
 L POWER_GND #03
 U 1 1 530346AA
-P 6100 3850
-F 0 "#03" V 6050 3800 60  0001 C CNN
-F 1 "POWER_GND" V 6150 3800 60  0001 C CNN
-F 2 "" H 6100 3850 60  0000 C CNN
-F 3 "" H 6100 3850 60  0000 C CNN
-	1    6100 3850
+P 7000 4550
+F 0 "#03" V 6950 4500 60  0001 C CNN
+F 1 "POWER_GND" V 7050 4500 60  0001 C CNN
+F 2 "" H 7000 4550 60  0000 C CNN
+F 3 "" H 7000 4550 60  0000 C CNN
+	1    7000 4550
 	1    0    0    -1
 $EndComp
@@
 L DIODE_LIGHT VD1
 U 1 1 5303476E
-P 5250 3650
-F 0 "VD1" H 5600 3950 60  0000 C CNN
-F 1 "DIODE_LIGHT" H 5600 3400 60  0000 C CNN
-F 2 "" H 5250 3650 60  0000 C CNN
-F 3 "" H 5250 3650 60  0000 C CNN
-	1    5250 3650
+P 6100 3100
+F 0 "VD1" V 6100 3300 60  0000 C CNN
+F 1 "DIODE_LIGHT" H 6450 2850 60  0001 C CNN
+F 2 "" H 6100 3100 60  0000 C CNN
+F 3 "" H 6100 3100 60  0000 C CNN
+	1    6100 3100
 	0    -1   1    0
 $EndComp
@@
 L PWR_FLAG #FLG06
 U 1 1 53038977
-P 4900 2750
-F 0 "#FLG06" H 4900 2845 30  0001 C CNN
-F 1 "PWR_FLAG" H 4900 2930 30  0000 C CNN
-F 2 "" H 4900 2750 60  0000 C CNN
-F 3 "" H 4900 2750 60  0000 C CNN
-	1    4900 2750
+P 5750 2750
+F 0 "#FLG06" H 5750 2845 30  0001 C CNN
+F 1 "PWR_FLAG" H 5750 3000 30  0000 C CNN
+F 2 "" H 5750 2750 60  0000 C CNN
+F 3 "" H 5750 2750 60  0000 C CNN
+	1    5750 2750
 	1    0    0    -1
 $EndComp
@@
 P 7250 2650
 F 0 "DA1" H 7750 2800 60  0000 C CNN
-F 1 "УД608" H 7750 2100 60  0000 C CNN
+F 1 "УД608" H 7750 2050 60  0000 C CNN
 F 2 "~" H 7250 2650 60  0000 C CNN
 F 3 "~" H 7250 2650 60  0000 C CNN
@@
 	7150 2650 7150 2100
 Wire Wire Line
-	6200 2100 5750 2100
+	6200 2100 5100 2100
 Wire Wire Line
 	7050 2850 7250 2850
@@
 Connection ~ 7150 2850
 Wire Wire Line
-	6200 3650 6100 3650
-Wire Wire Line
-	6100 3650 6100 3850
-Wire Wire Line
-	4550 4350 4550 4250
-Wire Wire Line
-	4550 4800 4550 5700
-Connection ~ 4550 3500
-Wire Wire Line
-	4550 2850 6250 2850
-Connection ~ 5250 2850
+	7000 4500 7000 4550
+Wire Wire Line
+	5400 3800 5400 3700
+Wire Wire Line
+	5400 2850 6250 2850
 Wire Wire Line
 	8250 3050 8400 3050
@@
 Connection ~ 8650 2650
 Wire Wire Line
-	4550 3150 4550 3850
-Wire Wire Line
-	4550 3050 4550 2850
-Wire Wire Line
-	5250 4450 5250 4250
+	6100 3900 6100 3700
 Wire Wire Line
 	6650 2100 7350 2100
@@
 	8250 2850 8400 2850
 Wire Wire Line
-	8400 2850 8400 2350
-Wire Wire Line
-	8400 2350 5250 2350
-Wire Wire Line
-	5250 2350 5250 3650
-Wire Wire Line
-	4900 2750 4900 2850
-Connection ~ 4900 2850
+	8400 2850 8400 2400
+Wire Wire Line
+	5750 2750 5750 2850
+Connection ~ 5750 2850
 Wire Wire Line
 	8900 3700 8900 3850
-Wire Wire Line
-	5250 5600 5250 5250
-Connection ~ 4550 5400
-Connection ~ 4550 5600
-Wire Wire Line
-	4350 5400 4550 5400
+Connection ~ 5400 4500
+Connection ~ 5400 4700
+Wire Wire Line
+	5200 4500 5400 4500
 $Comp
 L PWR_FLAG #FLG07
 U 1 1 530388A3
-P 4350 5400
-F 0 "#FLG07" H 4350 5495 30  0001 C CNN
-F 1 "PWR_FLAG" H 4350 5580 30  0000 C CNN
-F 2 "" H 4350 5400 60  0000 C CNN
-F 3 "" H 4350 5400 60  0000 C CNN
-	1    4350 5400
-	1    0    0    -1
-$EndComp
-Wire Wire Line
-	5250 5600 4550 5600
+P 5200 4500
+F 0 "#FLG07" H 5200 4595 30  0001 C CNN
+F 1 "PWR_FLAG" H 5200 4750 30  0000 C CNN
+F 2 "" H 5200 4500 60  0000 C CNN
+F 3 "" H 5200 4500 60  0000 C CNN
+	1    5200 4500
+	1    0    0    -1
+$EndComp
+Wire Wire Line
+	5400 4700 6100 4700
 $Comp
 L BUZZER BZ1
 U 1 1 5303A8D4
 P 9150 3600
-F 0 "BZ1" H 9050 3850 70  0000 C CNN
-F 1 "BUZZER" H 9050 3350 70  0000 C CNN
+F 0 "BZ1" H 9450 3600 70  0000 C CNN
+F 1 "BUZZER" H 9050 3350 70  0001 C CNN
 F 2 "~" H 9150 3600 60  0000 C CNN
 F 3 "~" H 9150 3600 60  0000 C CNN
@@
 Wire Wire Line
 	8900 3500 8900 3450
+Wire Wire Line
+	8400 2400 5400 2400
+Wire Wire Line
+	7000 3700 7000 3650
+Wire Wire Line
+	6100 3100 6100 2850
+Connection ~ 6100 2850
+Wire Wire Line
+	5400 3300 5400 3150
+Wire Wire Line
+	5400 4250 5400 4800
+Wire Wire Line
+	5400 2400 5400 3050
+Connection ~ 5400 2850
 $EndSCHEMATC

Commit message: next step
Parts:
- C1: value 0,1 -> 1,0мкФ
- R1: value 5,1K -> 820
- R3: value 1,8K -> 5,1K
Changed lines of the file:
@@
 P 7350 2100
 F 0 "R1" H 7600 2225 60  0000 C CNN
-F 1 "5,1K" H 7600 1950 60  0000 C CNN
+F 1 "820" H 7600 1950 60  0000 C CNN
 F 2 "" H 7350 2100 60  0000 C CNN
 F 3 "" H 7350 2100 60  0000 C CNN
@@
 P 7000 4500
 F 0 "R3" V 7600 4350 60  0000 C CNN
-F 1 "1,8K" V 7250 4250 60  0000 C CNN
+F 1 "5,1K" V 7250 4250 60  0000 C CNN
 F 2 "" H 7000 4500 60  0000 C CNN
 F 3 "" H 7000 4500 60  0000 C CNN
@@
 P 6200 2100
 F 0 "C1" V 6350 1750 60  0000 C CNN
-F 1 "0,1" V 6100 1750 60  0000 C CNN
+F 1 "1,0мкФ" V 6100 1650 60  0000 C CNN
 F 2 "" H 6200 2100 60  0000 C CNN
 F 3 "" H 6200 2100 60  0000 C CNN
